File: 25720-03 Power Supply/25720-03 Power Supply.kicad_sch (KiCad schematic)
At the start: 43 parts, among them T1 Transformer_1P_2S, U2 TNY180P

Commit message: small corrections
Parts:
- D201: value SR320D -> SR3200
- renumbered U2 to IC101
Connections:
- net +2V5: now reaches C204.2, IC201.3 (VCTRL), R207.2, R208.1, R208A1.1, R209.2
Other:
- moved on the sheet: EC101, EC102, F101, VR101

Commit message: minor changes
Other:
- title: 205720-03 power supply -> 205720-03 battery charger
Changed lines of the file:
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@@
 	(paper "A4")
 	(title_block
-		(title "205720-03 power supply")
+		(title "205720-03 battery charger")
 		(company "Dyson")
-		(comment 1 "26.1V, 0.78A")
 		(comment 2 "Manufacturer: Salom Electric")
+		(comment 3 "Input: 100-240V ~ 50/60Hz 0.6A")
+		(comment 4 "Output: 26.10V =, 0.78A")
 	)
 	(text "Secondary: Typical Application 1 Circuit of AP4320 (from datasheet)\nVout=Vref*(R1+R2)/R1 = 24.1V\nR2=R207=360k, R1=R208//R208A//(R209+R210) =~ 38k\nCurrent limit = Vsense/R210 = 50mV/64mOhm =~ 0.78A"
@@
 		)
 	)
+	(polyline
+		(pts
+			(xy 87.63 66.04) (xy 116.84 66.04)
+		)
+		(stroke
+			(width 1)
+			(type dash_dot)
+		)
+	)
 	(wire
 		(pts
@@
 		)
 	)
+	(polyline
+		(pts
+			(xy 87.63 21.59) (xy 87.63 66.04)
+		)
+		(stroke
+			(width 1)
+			(type dash_dot)
+		)
+	)
 	(wire
 		(pts
@@
 			(width 0)
 			(type default)
+		)
+	)
+	(polyline
+		(pts
+			(xy 116.84 66.04) (xy 116.84 170.18)
+		)
+		(stroke
+			(width 1)
+			(type dash_dot)
 		)
 	)
@@
 		(dnp no)
 		(property "Reference" "EC201"
-			(at 127 94.3609 0)
+			(at 130.556 91.44 0)
 			(effects
 				(font
@@
 		)
 		(property "Value" "330uF, 35V"
-			(at 127 96.9009 0)
-			(effects
-				(font
+			(at 130.556 93.98 0)
+			(effects
+				(font
